Commit message: many changes, currently working on launching script

File: nuric_wheelchair_model_02/urdf/wheelchair.constants.xacro (robot description, xacro)
@@ -11,5 +11,6 @@
    <xacro:macro name="caster_wheel_inertia" >
       <inertial>
-        <mass value="0.07" />
+        <!--<mass value="0.07" /> -->
+        <mass value="0.0003" />
         <origin xyz="0 0 0" />
         <inertia  ixx="0.001" ixy="0.0" ixz="0.0"
@@ -19,5 +20,6 @@
    <xacro:macro name="caster_hub_inertia" params="lr">
       <inertial>
-        <mass value="0.015" />
+        <!--<mass value="0.015" /> -->
+        <mass value="0.0003" />
         <origin xyz="${lr*-0.043126} 0.030993 0.053064" />
         <inertia  ixx="0.001" ixy="0.0" ixz="0.0"

File: nuric_wheelchair_model_02/urdf/wheelchair.hokuyo.xacro (robot description, xacro)
@@ -33,5 +33,5 @@
  </link>
 <gazebo reference="laser_joint">
-  <sensor type="ray" name="laser">
+  <sensor type="gpu_ray" name="laser">
     <pose>0 0 0 0 0 0</pose>
     <visualize>true</visualize>
@@ -57,5 +57,5 @@
       </noise>
     </ray>
-    <plugin name="gazebo_ros_laser_controller" filename="libgazebo_ros_laser.so">
+    <plugin name="gazebo_ros_laser_controller" filename="libgazebo_ros_gpu_laser.so">
       <gaussianNoise>0.005</gaussianNoise>
       <alwaysOn>true</alwaysOn>

File: nuric_wheelchair_model_02/urdf/wheelchair.kinect.xacro (robot description, xacro)
@@ -134,6 +134,6 @@
   <gazebo reference="camera_link">
     <sensor type="depth" name="camera">
-      <always_on>true</always_on>
-      <visualize>true</visualize>
+      <always_on>false</always_on>
+      <visualize>false</visualize>
       <camera>
         <horizontal_fov>1.047</horizontal_fov>
@@ -150,5 +150,5 @@
         </clip>
       </camera>
-      <plugin name="kinect_camera_controller" filename="libgazebo_ros_openni_kinect.so">
+      <!--<plugin name="kinect_camera_controller" filename="libgazebo_ros_openni_kinect.so">
         <baseline>0.1</baseline>
         <alwaysOn>true</alwaysOn>
@@ -172,5 +172,5 @@
         <focalLength>0</focalLength>
         <hackBaseline>0.07</hackBaseline>
-      </plugin>
+      </plugin>-->
     </sensor>
   </gazebo>
